File: hardware/solid_state_relay.kicad_pcb (KiCad board)
At the start: 2 copper layers, 19 x 33.4 mm, 13 parts, among them P1 CON-SENSOR, P2 TST, P3 TST, Q1 2N7002P, U1 M24C64, U2 DRILL, U3 DRILL

Commit message: drc check
Parts:
- added Fiducial_Mark: VAL**, kicad-libraries:Fiducial_Mark, F.Cu at (105.4, 81.4)
Changed lines of the file:
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@@
-(kicad_pcb (version 3) (host pcbnew "(2014-06-08 BZR 4933)-product")
+(kicad_pcb (version 4) (host pcbnew "(2015-03-18 BZR 5525)-product")
   (general
     (links 19)
     (no_connects 0)
-    (area 97.102369 48.594339 282.371482 165.089523)
+    (area 98.209499 49.309499 117.590501 83.090501)
     (thickness 1.6002)
     (drawings 18)
     (tracks 109)
     (zones 0)
-    (modules 13)
+    (modules 14)
     (nets 13)
   )
@@
   )
   (layers
-    (15 Vorderseite signal hide)
-    (0 Rückseite signal hide)
-    (16 B.Adhes user)
-    (17 F.Adhes user)
-    (18 B.Paste user)
-    (19 F.Paste user)
-    (20 B.SilkS user)
-    (21 F.SilkS user)
-    (22 B.Mask user hide)
-    (23 F.Mask user hide)
-    (24 Dwgs.User user)
-    (25 Cmts.User user)
-    (26 Eco1.User user)
-    (27 Eco2.User user)
-    (28 Edge.Cuts user)
+    (0 Vorderseite signal hide)
+    (31 Rückseite signal hide)
+    (32 B.Adhes user)
+    (33 F.Adhes user)
+    (34 B.Paste user)
+    (35 F.Paste user)
+    (36 B.SilkS user)
+    (37 F.SilkS user)
+    (38 B.Mask user hide)
+    (39 F.Mask user hide)
+    (40 Dwgs.User user)
+    (41 Cmts.User user)
+    (42 Eco1.User user)
+    (43 Eco2.User user)
+    (44 Edge.Cuts user)
   )
   (setup
@@
     (visible_elements FFFFFFBF)
     (pcbplotparams
-      (layerselection 284196865)
+      (layerselection 0x010fc_80000001)
       (usegerberextensions true)
       (excludeedgelayer true)
@@
       (xy 2.50444 -3.40868) (xy 2.50444 -3.31978) (xy 2.50444 -3.31978)) (layer B.SilkS) (width 0.00254))
   )
+  (module kicad-libraries:Fiducial_Mark (layer Vorderseite)
+    (at 105.4 81.4)
+    (attr smd)
+    (fp_text reference Fiducial_Mark (at 0 0) (layer F.SilkS) hide
+      (effects (font (size 0.127 0.127) (thickness 0.03302)))
+    )
+    (fp_text value VAL** (at 0 -0.29972) (layer F.SilkS) hide
+      (effects (font (size 0.127 0.127) (thickness 0.03302)))
+    )
+    (fp_circle (center 0 0) (end 1.15062 0) (layer Dwgs.User) (width 0.01016))
+    (pad 1 smd circle (at 0 0) (size 1.00076 1.00076) (layers Vorderseite F.Mask)
+      (clearance 0.65024))
+  )
   (gr_text + (at 107.1 78.9) (layer F.SilkS)
